File: Twinkies.kicad_sch (KiCad schematic)
At the start: 33 parts, among them J1 GPS u.fl, J2 Radio u.fl, SW1 RESET, U1 MAX-M8Q, U2 RFM95W, U3 MPU-6050, U4 TLV493D, U5 BME280

Commit message: 0.1 Schematic
Schematic as of Feb 25
Parts:
- removed U?: INA219AxD, Package_SO:SOIC-8_3.9x4.9mm_P1.27mm, symbol Analog_ADC:INA219AxD
- added BT2: CR1220, symbol Device:Battery_Cell
- added C10, C12, C16, C4, C9: 1uF, symbol Device:C_Small
- added C11: 470pF, symbol Device:C_Small
- added J3: UART_GPIO, symbol Connector:Conn_01x02_Female
- added J4: GPIO_SPI, symbol Connector:Conn_01x07_Female
- added J5: GPIO_I2C, symbol Connector:Conn_01x12_Female
- added J6: GPIO_SDCARD, symbol Connector:Conn_01x06_Female
- added Q1: Q_NPN, symbol Device:Q_NPN_BCE
- added R? (x2): 10k, symbol Device:R
- added R?: 0.62R, symbol Device:R
- added U7: LTC2990, Package_SO:MSOP-10_3x3mm_P0.5mm, symbol Sensor:LTC2990
- added U9: VEML7700-TT, XDCR_VEML7700-TT, symbol VEML7700-TT:VEML7700-TT
- added Y1: Crystal, symbol Device:Crystal
- gave numbers to parts that had none: 12
Connections:
- net RFM_MISO is gone; now on net BME_MISO: U2.2 (MISO)
- net RFM_MOSI is gone; now on net BME_MISO: U2.3 (MOSI)
- net RFM_SCK is gone; now on net BME_SCK: U2.4 (SCK)
- net +3V3: now also J1.3 (Pin_3), J2.4 (VDD), U3.9 (AD0), U5.6 (VDDIO), U5.8 (VDD), U6.8 (VDD), C10.2, C12.2, C16.2, C4.2, C9.2, R?.1, R?.1, R?.2, U7.1 (V1), U7.10 (VCC), U9.2; no longer C14.1
- net GND: now also J1.4 (Pin_4), J2.6 (VSS), J2.9 (SHIELD), U6.4 (VSS), BT2.2 (-), C10.1, C12.1, C16.1, C4.1, C9.1, U7.5 (GND), U7.8 (ADR0), U7.9 (ADR1), U9.3; no longer U3.9 (AD0)
- net GNSS_RX: now also J3.1 (Pin_1)
- net GNSS_TX: now also J3.2 (Pin_2)
- net IMU_SCL: now also J5.5 (Pin_5)
- net IMU_SDA: now also J5.6 (Pin_6)
- net MAG_SCL: now also J5.3 (Pin_3)
- net MAG_SDA: now also J5.4 (Pin_4)
- net RFM_CS: now also J4.2 (Pin_2)
- net RFM_RESET: now also J4.1 (Pin_1)
- net CAM_SCL: now reaches J1.1 (Pin_1)
- net CAM_SCL: now also J5.7 (Pin_7)
- net CAM_SDA: now reaches J1.2 (Pin_2)
- net CAM_SDA: now also J5.8 (Pin_8)
- net BME_SCK: now reaches J1.5 (Pin_5)
- net BME_SCK: now also U5.4 (SCK), J4.7 (Pin_7)
- net BME_MISO: now reaches J1.6 (Pin_6)
- net BME_MISO: now also J1.7 (Pin_7), J4.5 (Pin_5)
- net CAM_CS: now reaches J1.8 (Pin_8)
- net CAM_CS: now also J4.3 (Pin_3)
- net at U6.1 (OSCI): now also Y1.2
- net at U6.2 (OSCO): now also Y1.1
- net at U6.3 (VBAT): now also BT2.1 (+)
- net RTC_SDA: now reaches U6.5 (SDA)
- net RTC_SDA: now also J5.2 (Pin_2), R?.2
- net RTC_SCL: now reaches U6.6 (SCL)
- net RTC_SCL: now also J5.1 (Pin_1), R?.2
- net SDIO_DAT2: now reaches J2.1 (DAT2)
- net SDIO_DAT2: now also J6.1 (Pin_1)
- net SDIO_DAT3: now reaches J2.2 (DAT3/CD)
- net SDIO_DAT3: now also J6.2 (Pin_2)
- net SDIO_CMD: now reaches J2.3 (CMD)
- net SDIO_CMD: now also J6.3 (Pin_3)
- net SDIO_CLK: now reaches J2.5 (CLK)
- net SDIO_CLK: now also J6.4 (Pin_4)
- net SDIO_DAT0: now reaches J2.7 (DAT0)
- net SDIO_DAT0: now also J6.5 (Pin_5)
- net SDIO_DAT1: now reaches J2.8 (DAT1)
- net SDIO_DAT1: now also J6.6 (Pin_6)
- net BME_CS: now reaches U5.2 (CSB)
- net BME_CS: now also J4.4 (Pin_4)
- net BME_SDI: now reaches U5.3 (SDI)
- net BME_SDO: now reaches U5.5 (SDO)
- new net: C11.1, Q1.1 (B), Q1.2 (C), U7.3 (V3)
- new net: C11.2, Q1.3 (E), U7.4 (V4)
- new net 3V3_REG: C14.1, R?.1, U7.2 (V2)
- new net LTR_SCL: J5.9 (Pin_9), U9.1
- new net LTR_SDA: J5.10 (Pin_10), U9.4
- new net MISO: J4.6 (Pin_6)
- new net PWR_SCL: J5.11 (Pin_11), U7.7 (SCL)
- new net PWR_SDA: J5.12 (Pin_12), U7.6 (SDA)
- no-connect marks 13 -> 23
Other:
- note added: "Ambient light sensor: uses I2C, default addr = 0x10"
- note added: "External LNA for GNSS?"
- note added: "External LNA/PA?"
- note added: "GPIO Female Pins"
- note added: "Humidity + Barometric Pressure + Temperature Uses I2C or SPI, default addr = 0x77 Change to 0x76 by SDO<->GND"
- note added: "I/V measurement IC, Uses I2C Default addr = 0x98"
- note added: "IMU: uses I2C, default addr = 0x69 (AD0 to 3V3)"
- note added: "RTC, uses I2C, default addr = 0x68"
- note added: "SCK is I2C SCL SDI is I2C SDA SDO is MISO SDI is MOSI"
- note removed: "Humidity + Barometric Pressure + Temperature Uses I2C"
- note removed: "IMU: uses I2C, default addr = 0x68"
- note removed: "Power meter: Uses I2C, default addr ="
- moved on the sheet: BT1, C13, C14, C15, C2, C3, C5, C6, C7, C8, D1, J1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
