File: pdu.kicad_sch (KiCad schematic)
At the start: 24 parts

Commit message: Apr 8
Parts:
- removed C? (x3): 10uF, symbol Device:C_Small
- removed R? (x2): 250, Resistor_SMD:R_0603_1608Metric, symbol Device:R_Small
- removed U?: MAX8677AETG+T, 21-0139_T2444+4_MXM, symbol MAX8677AETG-T:MAX8677AETG+T
- removed U?: LTC4415EMSE#TRPBF, MSOP-16_MSE, symbol LTC4415EMSE_TRPBF:LTC4415EMSE#TRPBF
- added C14: 22uF, Capacitor_SMD:C_0603_1608Metric, symbol Device:C_Small
- added C16, C17: 10uF, Capacitor_SMD:C_0603_1608Metric, symbol Device:C_Small
- added C18: 470pF, Capacitor_SMD:C_0603_1608Metric, symbol Device:C_Small
- added C19: 4.7uF, Capacitor_SMD:C_0603_1608Metric, symbol Device:C_Small
- added C20, C21: 0.1uF, Capacitor_SMD:C_0603_1608Metric, symbol Device:C_Small
- added C22: 22nF, Capacitor_SMD:C_0603_1608Metric, symbol Device:C_Small
- added C23: 0.47uF, Capacitor_SMD:C_0603_1608Metric, symbol Device:C_Small
- added C24: 1nF, Capacitor_SMD:C_0603_1608Metric, symbol Device:C_Small
- added D2: D_Schottky, Diode_SMD:D_0603_1608Metric, symbol Device:D_Schottky
- added J6: PV_Jack, Connector_BarrelJack:BarrelJack_Horizontal, symbol Connector:Barrel_Jack
- added J9: Conn_Batt, Connector_JST:JST_PH_S2B-PH-SM4-TB_1x02-1MP_P2.00mm_Horizontal, symbol Connector_Generic:Conn_01x02
- added Q1: UMT3904T106, SOT65:SOT65P210X100-3N, symbol Device:Q_NPN_BCE
- added Q2, Q3: DMG3414U, Package_TO_SOT_SMD:SOT-23, symbol Transistor_FET:DMG3414U
- added R22: 1R, Resistor_SMD:R_0603_1608Metric, symbol Device:R
- added R23, R25, R30, R31: 4.7k, Resistor_SMD:R_0603_1608Metric, symbol Device:R_Small
- added R24: 10mR, Resistor_SMD:R_0603_1608Metric, symbol Device:R_Small
- added R26: 10R, Resistor_SMD:R_0603_1608Metric, symbol Device:R_Small
- added R27: 100R, Resistor_SMD:R_0603_1608Metric, symbol Device:R_Small
- added R28, R29: 1k, Resistor_SMD:R_0603_1608Metric, symbol Device:R_Small
- added R32: 10k, Resistor_SMD:R_0603_1608Metric, symbol Device:R_Small
- added U10: AZ1117H-5.0TRG1, Package_TO_SOT_SMD:SOT-223, symbol Regulator_Linear:AZ1117-3.3
- added U12: AZ1117-3.3, Package_TO_SOT_SMD:SOT-223, symbol Regulator_Linear:AZ1117-3.3
- added U13: LTC2990, Package_SO:MSOP-10_3x3mm_P0.5mm, symbol Sensor:LTC2990
- added U14: MAX17330X22+, MAX17330X22:MAX17330X22&plus_, symbol MAX17330X22:MAX17330X22+
- C10, C11, C12, C13, C15: renamed from C?; footprint (none) -> Capacitor_SMD:C_0603_1608Metric
- J7: renamed from J?; footprint (none) -> Connector_BarrelJack:BarrelJack_Horizontal
- L1: renamed from L?; footprint (none) -> Inductor_SMD:L_0603_1608Metric
- R14, R17, R18, R19, R20, R21: renamed from R?; footprint (none) -> Resistor_SMD:R_0603_1608Metric
- U11: renamed from U?; footprint SOP65P640X120-8N -> SPV1040T:SOP65P640X120-8N
- gave numbers to parts that had none: 3
Connections:
- net GND: now also C14.1, C16.2, C17.2, C19.2, C21.2, C23.2, C24.2, J6.2, J9.2 (Pin_2), U10.1 (GND), U12.1 (GND), U13.5 (GND), U13.8 (ADR0), U13.9 (ADR1), U14.A2 (GND)
- net V_DC: now also C14.2, U10.2 (VO); no longer C11.2, J7.1
- net at L1.1, U11.3 (LX): now also D2.2 (A)
- net at R18.2, R19.2, R21.1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: now also D2.1 (K)
- net PV+: no longer names the net of R14.1
- net PV+: now also J6.1
- net USB_D+ renamed USBPLUG_D+
- net USB_D- renamed USBPLUG_D-
- new net: Q2.1 (G), R27.2
- new net: C22.2, Q2.2 (S), R24.2, U14.A3 (CSP)
- new net: Q2.3 (D), Q3.3 (D)
- new net: C18.1, Q1.1 (B), Q1.2 (C), U13.3 (V3)
- new net: C18.2, Q1.3 (E), U13.4 (V4)
- new net: C22.1, R27.1, U14.C2 (CHG)
- new net: R28.1, U14.C3 (DIS)
- new net: Q3.1 (G), R28.2
- new net: C20.2, C21.1, R26.2, U14.A1 (TH), U14.C1 (BATT)
- new net: C19.1, J9.1 (Pin_1), R24.1, R26.1, U14.A4 (CSN)
- new net: C23.1, U14.A5 (REG)
- new net: C20.1, U14.B1 (CP)
- new net: C24.1, R29.1, U14.C4 (PCKP)
- new net: C11.2, J7.1, U10.3 (VI)
- new net +3V3: R22.2, R23.2, R25.2, R30.2, R31.2, R32.2, U13.1 (V1), U13.10 (VCC)
- new net 3V3_REG: C17.1, R22.1, U12.2 (VO), U13.2 (V2)
- new net BMIC_ALERT: R32.1, U14.B4 (ALRT/PIO)
- new net BMIC_SCL: R31.1, U14.B5 (SCL)
- new net BMIC_SDA: R30.1, U14.C5 (SDA)
- new net PWR_SCL: R25.1, U13.7 (SCL)
- new net PWR_SDA: R23.1, U13.6 (SDA)
- new net VBUS: C16.1, Q3.2 (S), R29.2, U12.3 (VI)
- no-connect marks 2 -> 4
Other:
- added sheet LTC4417 (ltc4417.kicad_sch)
- note added: "Battery charger, protector and SOC monitor"
- note added: "I/V measurement IC, Uses I2C Default addr = 0x98"
- note added: "VBUS = the highest of the 3 input powers"
- note removed: "Limit current to 2A"
- note removed: "Power MUX switch"
