File: sensors.kicad_sch (KiCad schematic)
At the start: 49 parts, among them J1 UART_GPIO, J2 Radio u.fl, J3 GPIO_SPI, J4 GPS u.fl, J5 GPIO_I2C, J6 GPIO_SDCARD, J7 USB-C Power, J8 Arducam, J9 Micro_SD_Card, Q1 Q_NPN, SW1 RESET, U1 RFM95W, U2 MAX-M8Q, U3 MCP7940NT-I/MS, U4 VEML7700-TT, U5 TLV493D, U6 MPU-6050, U7 BME280, U8 LTC2990, U9 AP2112K-3.3, Y1 32.768kHz

Commit message: 3.4
Parts:
- removed C10: 1uF, Capacitor_SMD:C_0603_1608Metric, symbol Device:C_Small
- removed C13, C14: 10uF, Capacitor_SMD:C_0603_1608Metric, symbol Device:C_Small
- removed C8: 0.1uF, Capacitor_SMD:C_0603_1608Metric, symbol Device:C_Small
- removed J1: UART_GPIO, symbol Connector:Conn_01x02_Female
- removed J3: GPIO_SPI, symbol Connector:Conn_01x07_Female
- removed J5: GPIO_I2C, symbol Connector:Conn_01x12_Female
- removed J6: GPIO_SDCARD, symbol Connector:Conn_01x06_Female
- removed J7: USB-C Power, symbol Connector:USB_C_Receptacle_USB2.0
- removed R10: 100k, Resistor_SMD:R_0603_1608Metric, symbol Device:R
- removed R6, R8: 10k, Resistor_SMD:R_0603_1608Metric, symbol Device:R
- removed U3: MCP7940NT-I/MS, symbol Timer_RTC:MCP7940N-xMS
- removed U6: MPU-6050, Sensor_Motion:InvenSense_QFN-24_4x4mm_P0.5mm, symbol Sensor_Motion:MPU-6050
- removed U9: AP2112K-3.3, Package_TO_SOT_SMD:SOT-23-5, symbol Regulator_Linear:AP2112K-3.3
- added J1: Conn_01x12, Connector_PinHeader_2.54mm:PinHeader_1x13_P2.54mm_Vertical, symbol Connector_Generic:Conn_01x12
- added J3: Conn_01x06, Connector_PinHeader_2.54mm:PinHeader_1x06_P2.54mm_Vertical, symbol Connector_Generic:Conn_01x06
- added J5: Conn_01x18, Connector_PinHeader_2.54mm:PinHeader_1x18_P2.54mm_Vertical, symbol Connector_Generic:Conn_01x18
- added U3: DS1339BU+T, DS1339BU_T:SOP65P490X110-8N, symbol DS1339BU_T:DS1339BU+T
- added U6: PCA9548AD,118, PCA9548AD_118:SOIC127P1032X265-24N, symbol Interface_Expansion:PCA9548ADW
- added U9: ISM330DHCXTR, ISM330DHCXTR:LGA-14_2.5X3X0.86_, symbol ISM330DHCXTR:ISM330DHCXTR
- BT1: footprint BAT_S8411-45R -> S8411-45R:BAT_S8411-45R
- C7: value 2.2nF -> 1uF
- J8: footprint (none) -> Connector_PinHeader_2.54mm:PinHeader_1x18_P2.54mm_Vertical
- J9: value Micro_SD_Card -> DM3AT-SF-PEJM5; footprint (none) -> DM3AT-SF-PEJM5:HRS_DM3AT-SF-PEJM5
- Q1: value Q_NPN -> UMT3904T106; footprint (none) -> SOT65:SOT65P210X100-3N
- U1: footprint (none) -> RFM95W-915S2:XCVR_RFM95W-915S2
- Y1: footprint (none) -> eec:Abracon-ABS07-120-0-0-MFG
Connections:
- net 3V3_REG is gone; now on net +3V3: R11.1, U8.2 (V2)
- net CAM_MISO is gone; now on net BME_SDO: J8.6 (Pin_6)
- net CAM_MOSI is gone; now on net BME_SDI: J8.7 (Pin_7)
- net CAM_SCK is gone; now on net BME_SCK: J8.5 (Pin_5)
- net RFM_MISO is gone; now on net BME_SDO: U1.2 (MISO)
- net RFM_MOSI is gone; now on net BME_SDI: U1.3 (MOSI)
- net RFM_SCK is gone; now on net BME_SCK: U1.4 (SCK)
- net +3V3: now also C7.2, U3.8 (VCC), U6.24 (VCC), U9.5 (VDDIO), U9.8 (VDD)
- net BME_CS: now also J5.11 (Pin_11)
- net BME_SCK: now also J5.12 (Pin_12), J5.4 (Pin_4), J5.9 (Pin_9)
- net BME_SDI: now also J5.14 (Pin_14), J5.5 (Pin_5), J5.8 (Pin_8)
- net BME_SDO: now also J5.10 (Pin_10), J5.13 (Pin_13), J5.6 (Pin_6)
- net CAM_CS: now also J5.15 (Pin_15)
- net CAM_SCL: now also J1.7 (Pin_7), U6.11 (SC3)
- net CAM_SDA: now also J1.8 (Pin_8), U6.10 (SD3)
- net GND: now also C7.1, U3.4 (GND), U6.1 (A0), U6.12 (GND), U6.2 (A1), U6.21 (A2), U9.2 (SDX), U9.3 (SCX), U9.6 (GND_1), U9.7 (GND_2); no longer C7.2
- net GNSS_RX: now also J5.1 (Pin_1)
- net GNSS_TX: now also J5.2 (Pin_2)
- net IMU_SCL: now also J1.5 (Pin_5), U6.9 (SC2), U9.14 (SDA)
- net IMU_SDA: now also J1.6 (Pin_6), U6.8 (SD2), U9.13 (SCL)
- net LTR_SCL: now also J1.9 (Pin_9), U6.14 (SC4)
- net LTR_SDA: now also J1.10 (Pin_10), U6.13 (SD4)
- net MAG_SCL: now also J1.3 (Pin_3), U6.7 (SC1)
- net MAG_SDA: now also J1.4 (Pin_4), U6.6 (SD1)
- net PWR_SCL: now also J1.11 (Pin_11), U6.16 (SC5)
- net PWR_SDA: now also J1.12 (Pin_12), U6.15 (SD5)
- net RFM_CS: now also J5.7 (Pin_7)
- net RFM_RESET: now also J5.3 (Pin_3)
- net RTC_BCKP: now also U3.3 (VBACKUP)
- net RTC_SCL: now also J1.1 (Pin_1), U3.6 (SCL), U6.5 (SC0)
- net RTC_SDA: now also J1.2 (Pin_2), U3.5 (SDA), U6.4 (SD0)
- net SDIO_CLK: now also J3.4 (Pin_4)
- net SDIO_CMD: now also J3.3 (Pin_3)
- net SDIO_DAT0: now also J3.5 (Pin_5)
- net SDIO_DAT1: now also J3.6 (Pin_6)
- net SDIO_DAT2: now also J3.1 (Pin_1)
- net SDIO_DAT3: now also J3.2 (Pin_2)
- net at Y1.1: now also U3.2 (X2)
- net at Y1.2: now also U3.1 (X1)
- new net IMU_CS: J5.16 (Pin_16), U9.12 (CS)
- new net IMU_INT1: J5.17 (Pin_17), U9.4 (INT1)
- new net IMU_INT2: J5.18 (Pin_18), U9.9 (INT2)
- new net IMU_MISO: U9.1 (SDO/SA0)
- new net MUX_SCL: U6.22 (SCL)
- new net MUX_SDA: U6.23 (SDA)
- no-connect marks 22 -> 13
Other:
- note added: "Debug Headers"
- note added: "IMU: uses I2C, default addr = 0x6a"
- note removed: "3v3 regulator"
- note removed: "External LNA for GNSS?"
- note removed: "GPIO Female Pins for debug"
- note removed: "IMU: uses I2C, default addr = 0x69 (AD0 to 3V3)"
- moved on the sheet: BT1, C1, C15, C3, C4, J2, J8, R4, R5, U1, U4, U7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

Commit message: 3/6
Parts:
- removed C7: 1uF, Capacitor_SMD:C_0603_1608Metric, symbol Device:C_Small
- removed J1: Conn_01x12, Connector_PinHeader_2.54mm:PinHeader_1x13_P2.54mm_Vertical, symbol Connector_Generic:Conn_01x12
- removed J5: Conn_01x18, Connector_PinHeader_2.54mm:PinHeader_1x18_P2.54mm_Vertical, symbol Connector_Generic:Conn_01x18
- removed U6: PCA9548AD,118, PCA9548AD_118:SOIC127P1032X265-24N, symbol Interface_Expansion:PCA9548ADW
- added C8: 100nF, Capacitor_SMD:C_0603_1608Metric, symbol Device:C_Small
- added J5: I2C, Connector_PinSocket_2.54mm:PinSocket_1x16_P2.54mm_Vertical, symbol Connector_Generic:Conn_01x16
- added J7: UART+SPI, Connector_PinSocket_2.54mm:PinSocket_1x11_P2.54mm_Vertical, symbol Connector_Generic:Conn_01x11
- added R11, R12, R4, R6: 10k, Resistor_SMD:R_0603_1608Metric, symbol Device:R
- added R15, R16: 4.7k, Resistor_SMD:R_0603_1608Metric, symbol Device:R
- J6: renamed from J8; footprint Connector_PinHeader_2.54mm:PinHeader_1x18_P2.54mm_Vertical -> Connector_PinHeader_2.54mm:PinHeader_1x08_P2.54mm_Vertical
- J8: renamed from J3; value Conn_01x06 -> SDIO
- R17: renamed from R11; value 0.62R -> 1
- renumbered C9 to C10, C15 to C12, C12 to C13, C1 to C3, C3 to C4, C2 to C5, C4 to C6, C5 to C7, C6 to C9, D1 to D2, J4 to J3, J9 to J4, R3 to R10, R7 to R13, R9 to R14, R4 to R5, R5 to R7, R1 to R8, R2 to R9, SW1 to SW3, U8 to U10, U1 to U3, U2 to U4, U3 to U5, U9 to U6, U4 to U7, U5 to U8, U7 to U9
Connections:
- net BME_CS is gone; now on net +3V3: U9.2 (CSB)
- net IMU_CS is gone; now on net +3V3: U6.12 (CS)
- net IMU_MISO is gone; now on net GND: U6.1 (SDO/SA0)
- net RTC_BCKP is gone; now on net +BATT: U5.3 (VBACKUP)
- net +3V3: now also C8.2, R11.1, R12.1, R15.1, R16.1, R4.1, R6.1
- net CAM_CS: now also J7.11 (Pin_11)
- net CAM_SCL: now also J5.6 (Pin_6)
- net CAM_SDA: now also J5.5 (Pin_5)
- net GND: now also U9.5 (SDO), C8.1
- net GNSS_RX: now also J7.1 (Pin_1)
- net GNSS_TX: now also J7.2 (Pin_2)
- net IMU_SCL: now also U6.13 (SCL), J5.8 (Pin_8), R12.2; no longer U6.14 (SDA)
- net IMU_SDA: now also U6.14 (SDA), J5.7 (Pin_7), R11.2; no longer U6.13 (SCL)
- net LTR_SCL: now also J5.4 (Pin_4)
- net LTR_SDA: now also J5.3 (Pin_3)
- net MAG_SCL: now also J5.10 (Pin_10)
- net MAG_SDA: now also J5.9 (Pin_9)
- net PWR_SCL: now also J5.2 (Pin_2)
- net PWR_SDA: now also J5.1 (Pin_1)
- net RFM_CS: now also J7.7 (Pin_7)
- net RFM_RESET: now also J7.3 (Pin_3)
- net RTC_SCL: now also J5.12 (Pin_12)
- net RTC_SDA: now also J5.11 (Pin_11)
- net TIMEPULSE: now also D2.2 (A)
- net GNSS_SDA: now reaches U4.16 (SDA)
- net GNSS_SDA: now also J5.13 (Pin_13), R4.2
- net GNSS_SCL: now reaches U4.17 (SCL)
- net GNSS_SCL: now also J5.14 (Pin_14), R6.2
- removed net BME_SCK: J6.5 (Pin_5), U3.4 (SCK), U9.4 (SCK)
- removed net BME_SDI: J6.7 (Pin_7), U3.3 (MOSI), U9.3 (SDI)
- removed net BME_SDO: J6.6 (Pin_6), U3.2 (MISO), U9.5 (SDO)
- net GNSS_BCKP renamed +BATT
- net IMU_INT1: no longer names the net of U6.4 (INT1)
- net IMU_INT2: no longer names the net of U6.9 (INT2)
- new net BME_SCL: J5.16 (Pin_16), R16.2, U9.4 (SCK)
- new net BME_SDA: J5.15 (Pin_15), R15.2, U9.3 (SDI)
- new net CAM_MISO: J6.6 (Pin_6), J7.9 (Pin_9)
- new net CAM_MOSI: J6.7 (Pin_7), J7.10 (Pin_10)
- new net CAM_SCK: J6.5 (Pin_5), J7.8 (Pin_8)
- new net RFM_MISO: J7.6 (Pin_6), U3.2 (MISO)
- new net RFM_MOSI: J7.5 (Pin_5), U3.3 (MOSI)
- new net RFM_SCK: J7.4 (Pin_4), U3.4 (SCK)
- no-connect marks 13 -> 16
Other:
- note added: "CS pulled high to lock into I2C mode"
- note added: "CSB pulled high to lock in I2C"
- note added: "Humidity + Barometric Pressure + Temperature Uses I2C, default addr = 0x77"
- note added: "Pin and footprint compatible with MAX-7"
- note removed: "Humidity + Barometric Pressure + Temperature Uses I2C or SPI, default addr = 0x77 Change to 0x76 by SDO<->GND"
- note removed: "SCK is I2C SCL SDI is I2C SDA SDO is MISO SDI is MOSI"
- moved on the sheet: BT1, C5, D2, J3, J6, J8, R10, R8, R9, SW3, U4

Commit message: pdu design
Parts:
- removed J5: I2C, Connector_PinSocket_2.54mm:PinSocket_1x16_P2.54mm_Vertical, symbol Connector_Generic:Conn_01x16
- removed J7: UART+SPI, Connector_PinSocket_2.54mm:PinSocket_1x11_P2.54mm_Vertical, symbol Connector_Generic:Conn_01x11
- removed J8: SDIO, Connector_PinHeader_2.54mm:PinHeader_1x06_P2.54mm_Vertical, symbol Connector_Generic:Conn_01x06
- removed U5: DS1339BU+T, DS1339BU_T:SOP65P490X110-8N, symbol DS1339BU_T:DS1339BU+T
- removed Y1: 32.768kHz, eec:Abracon-ABS07-120-0-0-MFG, symbol Device:Crystal
- added U?: RV-8523-C3, Package_SON:RTC_SMD_MicroCrystal_C3_2.5x3.7mm, symbol Timer_RTC:RV-8523-C3
Connections:
- net +3V3: now also U?.1 (VDD); no longer U3.13 (3.3V), U4.7 (VCC_IO), U4.8 (VCC)
- net +BATT: now also U?.8 (VBACKUP)
- net GND: now also U?.7 (VSS)
- net RTC_SCL: now also R7.2, U?.3 (SCL); no longer R5.2
- net RTC_SDA: now also R5.2, U?.4 (SDA); no longer R7.2
- new net GNSS_3V3: U4.7 (VCC_IO), U4.8 (VCC)
- new net RFM_3V3: U3.13 (3.3V)
- new net RTC_INT: U?.2 (~{INT_1})
- no-connect marks 16 -> 17
Other:
- note removed: "Debug Headers"
- note removed: "RTC, uses I2C, default addr = ?"
- moved on the sheet: C3, C4, D2, J6, R5, R7

Commit message: Apr 8
Parts:
- removed C11: 1uF, Capacitor_SMD:C_0603_1608Metric, symbol Device:C_Small
- removed C13: 470pF, Capacitor_SMD:C_0603_1608Metric, symbol Device:C_Small
- removed Q1: UMT3904T106, SOT65:SOT65P210X100-3N, symbol Device:Q_NPN_BCE
- removed R17: 1, Resistor_SMD:R_0603_1608Metric, symbol Device:R
- removed U10: LTC2990, Package_SO:MSOP-10_3x3mm_P0.5mm, symbol Sensor:LTC2990
- added U1, U5: TPS22902BYFPR, TPS22902BYFPR:TPS22902BYFPR, symbol TPS22902BYFPR:TPS22902BYFPR
- gave numbers to parts that had none: 1
- renumbered C3 to C1, C4 to C2, C5 to C3, C6 to C4, C7 to C5, C8 to C6, C9 to C7, C10 to C8, C12 to C9, D2 to D1, J6 to J5, R4 to R1, R13 to R10, R14 to R11, R15 to R12, R16 to R13, R6 to R2, R5 to R3, R8 to R4, R9 to R5, R7 to R6, R10 to R7, R11 to R8, R12 to R9, SW3 to SW1, U3 to U2
Connections:
- net +3V3: now also U1.A2 (VIN), U5.A2 (VIN)
- net GND: now also U1.B1 (GND), U5.B1 (GND)
- net GNSS_3V3: now also U5.A1 (VOUT)
- net RFM_3V3: now also U1.A1 (VOUT)
- new net GNSS_EN: U5.B2 (ON)
- new net RFM_EN: U1.B2 (ON)
- no-connect marks 17 -> 16
Other:
- note removed: "I/V measurement IC, Uses I2C Default addr = 0x98"
